File: hardware/Smart-Metering/02_Voltage_Sensing.kicad_sch (KiCad schematic)
At the start: 0 parts

Commit message: Implementa front-ends de tensão e corrente do ADE9430
02_Voltage_Sensing (3 fases, pseudo-diferencial):
- borne J101 (VA/VB/VC/VN) com labels globais LINE_A/B/C e NEUTRAL;
- fusível + varistor 320 VAC fase-neutro por fase;
- divisor 5 x 200 kΩ + 1 kΩ (1/1001): 220 V -> 0,311 Vpk, até ~354 Vrms
  com no máximo 0,5 Vpk por pino (limite do ADE9430: ±0,6 V);
- anti-aliasing 999 Ω // 22 nF (fc ≈ 7,2 kHz); VxN com 1 kΩ // 22 nF
  para casar impedância;
- R101 (0 Ω) liga NEUTRAL ao GND metrológico em ponto único.

03_Current_Sensing (IA/IB/IC/IN):
- entrada de TC por borne de 2 vias, TVS bidirecional SMAJ5.0CA;
- burden 2 x 10 Ω com center-tap no GND (TC 2500:1 -> fundo de escala
  ≈ 88 Arms, ±0,5 Vpk por pino);
- anti-aliasing 1 kΩ + 22 nF por perna (fc ≈ 7,2 kHz, casado com a tensão).

Biblioteca: novos símbolos Fuse, Varistor, D_TVS_Bi e
Screw_Terminal_01x02/01x04, já na convenção Y para cima do KiCad.

Co-Authored-By: Claude Opus 5.5 <noreply@anthropic.com>
Claude-Session: https://claude.ai/code/session_012B8cVkhtjf3eg98UdpNCpf
Parts:
- added C111, C112, C121, C122, C131, C132: 22nF C0G, Capacitor_SMD:C_0603_1608Metric, symbol SmartMetering:C_Vert
- added F101, F102, F103: 500mA 500VAC, symbol SmartMetering:Fuse
- added J101: VA VB VC VN, TerminalBlock_Phoenix:TerminalBlock_Phoenix_MKDS-1,5-4-5.08_1x04_P5.08mm_Horizontal, symbol SmartMetering:Screw_Terminal_01x04
- added R101: 0R, Resistor_SMD:R_1206_3216Metric, symbol SmartMetering:R_Vert
- added R111, R112, R113, R114, R115, R121, R122, R123, R124, R125, R131, R132, R133, R134, R135: 200k 0.1%, Resistor_SMD:R_1206_3216Metric, symbol SmartMetering:R_Vert
- added R116, R117, R126, R127, R136, R137: 1k 0.1%, Resistor_SMD:R_0603_1608Metric, symbol SmartMetering:R_Vert
- added RV101, RV102, RV103: 320VAC 14mm, symbol SmartMetering:Varistor
Connections:
- new net: R113.2, R114.1
- new net: R114.2, R115.1
- new net: R121.2, R122.1
- new net: R122.2, R123.1
- new net: F103.2, R131.1, RV103.1
- new net: R133.2, R134.1
- new net: R134.2, R135.1
- new net: R123.2, R124.1
- new net: R124.2, R125.1
- new net: R131.2, R132.1
- new net: R132.2, R133.1
- new net: F101.2, R111.1, RV101.1
- new net: R111.2, R112.1
- new net: F102.2, R121.1, RV102.1
- new net: R112.2, R113.1
- new net GND: C111.2, C112.2, C121.2, C122.2, C131.2, C132.2, R101.2, R116.2, R117.2, R126.2, R127.2, R136.2, R137.2
- new net LINE_A: F101.1, J101.1
- new net LINE_B: F102.1, J101.2
- new net LINE_C: F103.1, J101.3
- new net NEUTRAL: J101.4, R101.1, RV101.2, RV102.2, RV103.2
- new net VAN: C112.1, R117.1
- new net VAP: C111.1, R115.2, R116.1
- new net VBN: C122.1, R127.1
- new net VBP: C121.1, R125.2, R126.1
- new net VCN: C132.1, R137.1
- new net VCP: C131.1, R135.2, R136.1
Other:
- note added: "ENTRADA DE TENSÃO J101: 1 = VA, 2 = VB, 3 = VC, 4 = VN LINE_x/NEUTRAL são globais: 01_Power_Input pode derivar a alimentação daqui."
- note added: "FRONT-END DE TENSÃO — 3 FASES, PSEUDO-DIFERENCIAL Divisor: 5 x 200 kΩ + 1 kΩ -> atenuação 1/1001 220 Vrms -> 0,220 Vrms (0,311 Vpk) em VxP Limite por pino do ADE9430: ±0,6 V. Projeto: ≤ 0,5 Vpk -> Vmax ≈ 354 Vrms (1,6 x 220 V) Anti-aliasing: 999 Ω // 22 nF -> fc ≈ 7,2 kHz (igual aos canais de corrente) VxN: 1 kΩ // 22 nF para GND, casando a impedância vista por VxP Proteção por fase: fusível ≥ 50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"
- note added: "PONTO ÚNICO NEUTRO -> GND METROLÓGICO R101 0 Ω: montar em 3F+N / 1F+N. Não montar em 3 fios sem neutro."
- company: (none) -> Smart-Metering
- title: (none) -> Voltage Sensing - ADE9430 Front-End

Commit message: Implementa folha de entrada de energia e numera referências por folha
01_Power_Input:
- modo padrão: LINE_A/B/C -> fusível -> diodo S1M em OU para o
  barramento HV, retorno no NEUTRAL via JP101; o instrumento segue
  alimentado com qualquer fase presente;
- modo auxiliar (J101, 100-240 VAC, com varistor): F104/D104/JP102,
  não montados por padrão; para rede 3 fios sem neutro;
- R101 fusível limita inrush, C101 4,7 uF/450 V no barramento;
- PS101 módulo AC/DC isolado 5 V / 2 A (ex.: IRM-10-5) gerando
  VIN_ACDC para a folha 09, referenciado a GND_SYS.

Referências renumeradas por folha para evitar colisões: folha 02 passa
a 2xx (R201 = ligação neutro/GND), folha 03 a 3xx e folha 04 a 4xx
(U401 = ADE9430).

Novos símbolos: D_Rect, CP_Vert, Jumper_2 e ACDC_Module.

Co-Authored-By: Claude Opus 5.5 <noreply@anthropic.com>
Claude-Session: https://claude.ai/code/session_012B8cVkhtjf3eg98UdpNCpf
Parts:
- removed C111, C112, C121, C122, C131, C132: 22nF C0G, Capacitor_SMD:C_0603_1608Metric, symbol SmartMetering:C_Vert
- removed F101, F102, F103: 500mA 500VAC, symbol SmartMetering:Fuse
- removed J101: VA VB VC VN, TerminalBlock_Phoenix:TerminalBlock_Phoenix_MKDS-1,5-4-5.08_1x04_P5.08mm_Horizontal, symbol SmartMetering:Screw_Terminal_01x04
- removed R101: 0R, Resistor_SMD:R_1206_3216Metric, symbol SmartMetering:R_Vert
- removed R111, R112, R113, R114, R115, R121, R122, R123, R124, R125, R131, R132, R133, R134, R135: 200k 0.1%, Resistor_SMD:R_1206_3216Metric, symbol SmartMetering:R_Vert
- removed R116, R117, R126, R127, R136, R137: 1k 0.1%, Resistor_SMD:R_0603_1608Metric, symbol SmartMetering:R_Vert
- removed RV101, RV102, RV103: 320VAC 14mm, symbol SmartMetering:Varistor
- added C211, C212, C221, C222, C231, C232: 22nF C0G, Capacitor_SMD:C_0603_1608Metric, symbol SmartMetering:C_Vert
- added F201, F202, F203: 500mA 500VAC, symbol SmartMetering:Fuse
- added J201: VA VB VC VN, TerminalBlock_Phoenix:TerminalBlock_Phoenix_MKDS-1,5-4-5.08_1x04_P5.08mm_Horizontal, symbol SmartMetering:Screw_Terminal_01x04
- added R201: 0R, Resistor_SMD:R_1206_3216Metric, symbol SmartMetering:R_Vert
- added R211, R212, R213, R214, R215, R221, R222, R223, R224, R225, R231, R232, R233, R234, R235: 200k 0.1%, Resistor_SMD:R_1206_3216Metric, symbol SmartMetering:R_Vert
- added R216, R217, R226, R227, R236, R237: 1k 0.1%, Resistor_SMD:R_0603_1608Metric, symbol SmartMetering:R_Vert
- added RV201, RV202, RV203: 320VAC 14mm, symbol SmartMetering:Varistor
Connections:
- net GND: now also C211.2, C212.2, C221.2, C222.2, C231.2, C232.2, R201.2, R216.2, R217.2, R226.2, R227.2, R236.2, R237.2
- net LINE_A: now also F201.1, J201.1
- net LINE_B: now also F202.1, J201.2
- net LINE_C: now also F203.1, J201.3
- net NEUTRAL: now also J201.4, R201.1, RV201.2, RV202.2, RV203.2
- net VAN: now also C212.1, R217.1
- net VAP: now also C211.1, R215.2, R216.1
- net VBN: now also C222.1, R227.1
- net VBP: now also C221.1, R225.2, R226.1
- net VCN: now also C232.1, R237.1
- net VCP: now also C231.1, R235.2, R236.1
- new net: F201.2, R211.1, RV201.1
- new net: F203.2, R231.1, RV203.1
- new net: R231.2, R232.1
- new net: R222.2, R223.1
- new net: R223.2, R224.1
- new net: R224.2, R225.1
- new net: R221.2, R222.1
- new net: F202.2, R221.1, RV202.1
- new net: R212.2, R213.1
- new net: R213.2, R214.1
- new net: R214.2, R215.1
- new net: R211.2, R212.1
- new net: R232.2, R233.1
- new net: R233.2, R234.1
- new net: R234.2, R235.1
Other:
- note added: "ENTRADA DE TENSÃO J201: 1 = VA, 2 = VB, 3 = VC, 4 = VN LINE_x/NEUTRAL são globais: 01_Power_Input pode derivar a alimentação daqui."
- note added: "PONTO ÚNICO NEUTRO -> GND METROLÓGICO R201 0 Ω: montar em 3F+N / 1F+N. Não montar em 3 fios sem neutro."
- note removed: "ENTRADA DE TENSÃO J101: 1 = VA, 2 = VB, 3 = VC, 4 = VN LINE_x/NEUTRAL são globais: 01_Power_Input pode derivar a alimentação daqui."
- note removed: "PONTO ÚNICO NEUTRO -> GND METROLÓGICO R101 0 Ω: montar em 3F+N / 1F+N. Não montar em 3 fios sem neutro."

Commit message: Revisão completa do esquemático e correções
Verificação automática sobre o netlist global (215 componentes, 176 nets):
sem pinos soltos, sem nets de alimentação sem fonte, sem saídas em
conflito e isolação íntegra (terras só se encontram nas barreiras
PS101, PS601, U601, U602 e U801).

Correções:
- footprint do ADE9430 inexistente na biblioteca KiCad trocado por
  QFN-40 6x6 (tamanho do pad exposto a confirmar);
- MISO do ADE9430 como tri-state (barramento compartilhado com MCP3204);
- PS101 com símbolo e footprint oficiais do IRM-10-5 (o símbolo genérico
  tinha AC/L e AC/N trocados);
- PWR_FLAG em HV_DC, HV_RTN, VBAT_RTC, VDDA, GND_485 e VIN_CHG;
- footprints para fusíveis, varistores, indutores e chave de energia;
- polarização de fail-safe opcional no RS-485 (R807/R808, DNP);
- notas de layout (retorno do AC/DC) e de firmware (VBUS no PA9).

Relatório com revisão por folha, orçamento de potência e pendências em
docs/REVISAO_ESQUEMATICO.md.

Co-Authored-By: Claude Opus 5.5 <noreply@anthropic.com>
Claude-Session: https://claude.ai/code/session_012B8cVkhtjf3eg98UdpNCpf
Parts:
- F201, F202, F203: footprint (none) -> Fuse:Fuseholder_Clip-5x20mm_Littelfuse_111_Inline_P20.00x5.00mm_D1.05mm_Horizontal
- RV201, RV202, RV203: footprint (none) -> Varistor:RV_Disc_D15.5mm_W4.5mm_P7.5mm
Changed lines of the file:
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@@
 		(property "Reference" "F201" (at 63.5 60.96 0) (effects (font (size 1.27 1.27))))
 		(property "Value" "500mA 500VAC" (at 63.5 66.04 0) (effects (font (size 1.27 1.27))))
-		(property "Footprint" "" (at 63.5 63.5 0) (effects (font (size 1.27 1.27)) (hide yes)))
+		(property "Footprint" "Fuse:Fuseholder_Clip-5x20mm_Littelfuse_111_Inline_P20.00x5.00mm_D1.05mm_Horizontal" (at 63.5 63.5 0) (effects (font (size 1.27 1.27)) (hide yes)))
 		(property "Datasheet" "" (at 63.5 63.5 0) (effects (font (size 1.27 1.27)) (hide yes)))
 		(property "Description" "Phase A voltage-sense fuse, fast, >=500 VAC" (at 63.5 63.5 0) (effects (font (size 1.27 1.27)) (hide yes)))
@@
 		(property "Reference" "RV201" (at 74.93 66.04 0) (effects (font (size 1.27 1.27)) (justify left)))
 		(property "Value" "320VAC 14mm" (at 74.93 68.58 0) (effects (font (size 1.27 1.27)) (justify left)))
-		(property "Footprint" "" (at 72.39 67.31 0) (effects (font (size 1.27 1.27)) (hide yes)))
+		(property "Footprint" "Varistor:RV_Disc_D15.5mm_W4.5mm_P7.5mm" (at 72.39 67.31 0) (effects (font (size 1.27 1.27)) (hide yes)))
 		(property "Datasheet" "" (at 72.39 67.31 0) (effects (font (size 1.27 1.27)) (hide yes)))
 		(property "Description" "Phase A MOV to neutral (e.g. S14K320)" (at 72.39 67.31 0) (effects (font (size 1.27 1.27)) (hide yes)))
@@
 		(property "Reference" "F202" (at 63.5 99.06 0) (effects (font (size 1.27 1.27))))
 		(property "Value" "500mA 500VAC" (at 63.5 104.14 0) (effects (font (size 1.27 1.27))))
-		(property "Footprint" "" (at 63.5 101.6 0) (effects (font (size 1.27 1.27)) (hide yes)))
+		(property "Footprint" "Fuse:Fuseholder_Clip-5x20mm_Littelfuse_111_Inline_P20.00x5.00mm_D1.05mm_Horizontal" (at 63.5 101.6 0) (effects (font (size 1.27 1.27)) (hide yes)))
 		(property "Datasheet" "" (at 63.5 101.6 0) (effects (font (size 1.27 1.27)) (hide yes)))
 		(property "Description" "Phase B voltage-sense fuse, fast, >=500 VAC" (at 63.5 101.6 0) (effects (font (size 1.27 1.27)) (hide yes)))
@@
 		(property "Reference" "RV202" (at 74.93 104.14 0) (effects (font (size 1.27 1.27)) (justify left)))
 		(property "Value" "320VAC 14mm" (at 74.93 106.68 0) (effects (font (size 1.27 1.27)) (justify left)))
-		(property "Footprint" "" (at 72.39 105.41 0) (effects (font (size 1.27 1.27)) (hide yes)))
+		(property "Footprint" "Varistor:RV_Disc_D15.5mm_W4.5mm_P7.5mm" (at 72.39 105.41 0) (effects (font (size 1.27 1.27)) (hide yes)))
 		(property "Datasheet" "" (at 72.39 105.41 0) (effects (font (size 1.27 1.27)) (hide yes)))
 		(property "Description" "Phase B MOV to neutral (e.g. S14K320)" (at 72.39 105.41 0) (effects (font (size 1.27 1.27)) (hide yes)))
@@
 		(property "Reference" "F203" (at 63.5 137.16 0) (effects (font (size 1.27 1.27))))
 		(property "Value" "500mA 500VAC" (at 63.5 142.24 0) (effects (font (size 1.27 1.27))))
-		(property "Footprint" "" (at 63.5 139.7 0) (effects (font (size 1.27 1.27)) (hide yes)))
+		(property "Footprint" "Fuse:Fuseholder_Clip-5x20mm_Littelfuse_111_Inline_P20.00x5.00mm_D1.05mm_Horizontal" (at 63.5 139.7 0) (effects (font (size 1.27 1.27)) (hide yes)))
 		(property "Datasheet" "" (at 63.5 139.7 0) (effects (font (size 1.27 1.27)) (hide yes)))
 		(property "Description" "Phase C voltage-sense fuse, fast, >=500 VAC" (at 63.5 139.7 0) (effects (font (size 1.27 1.27)) (hide yes)))
@@
 		(property "Reference" "RV203" (at 74.93 142.24 0) (effects (font (size 1.27 1.27)) (justify left)))
 		(property "Value" "320VAC 14mm" (at 74.93 144.78 0) (effects (font (size 1.27 1.27)) (justify left)))
-		(property "Footprint" "" (at 72.39 143.51 0) (effects (font (size 1.27 1.27)) (hide yes)))
+		(property "Footprint" "Varistor:RV_Disc_D15.5mm_W4.5mm_P7.5mm" (at 72.39 143.51 0) (effects (font (size 1.27 1.27)) (hide yes)))
 		(property "Datasheet" "" (at 72.39 143.51 0) (effects (font (size 1.27 1.27)) (hide yes)))
 		(property "Description" "Phase C MOV to neutral (e.g. S14K320)" (at 72.39 143.51 0) (effects (font (size 1.27 1.27)) (hide yes)))
