File: hardware/Smart-Metering/02_Voltage_Sensing.kicad_sch (KiCad schematic)
At the start: 0 parts

Commit message: Alterações locais: folha 10 e ajustes nas folhas
Parts:
- added C20, C21, C22, C23, C24, C25: 22nF C0G 5%, Capacitor_SMD:C_0805_2012Metric, symbol SmartMetering:C_Vert
- added R20, R21, R22, R25, R26, R27, R30, R31, R32: 330k 0.1%, Resistor_SMD:R_1206_3216Metric, symbol SmartMetering:R_Vert
- added R23, R24, R28, R29, R33, R34: 1k 0.1%, Resistor_SMD:R_0603_1608Metric, symbol SmartMetering:R_Vert
Connections:
- new net: R20.1, R21.2
- new net: R21.1, R22.2
- new net: R25.1, R26.2
- new net: R26.1, R27.2
- new net: R30.1, R31.2
- new net: R31.1, R32.2
- new net GND: C20.1, C21.1, C22.1, C23.1, C24.1, C25.1, R23.1, R24.2, R28.1, R29.2, R33.1, R34.2
- new net PHASE_A_SENSE: R20.2
- new net PHASE_B_SENSE: R25.2
- new net PHASE_C_SENSE: R30.2
- new net VAN: C21.2, R24.1
- new net VAP: C20.2, R22.1, R23.2
- new net VBN: C23.2, R29.1
- new net VBP: C22.2, R27.1, R28.2
- new net VCN: C25.2, R34.1
- new net VCP: C24.2, R32.1, R33.2
Other:
- note added: "PHASE A"
- note added: "PHASE B"
- note added: "PHASE C"
- note added: "PRELIMINARY: 3P4W, 127/220 or 220/380 V, 60 Hz. VN_SENSE connects to metrology GND: mains-referenced domain. Divider 990k / 1k: ratio 1/991; voltage PGA = 1. RC nominal corner ~7.24 kHz. Calibrate including ADC loading. Input connectors, surge protection and isolation are NOT complete. Not approved for direct mains connection. 3-wire operation requires a separately validated reference strategy."
- company: (none) -> Smart-Metering
- title: (none) -> Voltage sensing - preliminary 3P4W
Changed lines of the file:
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@@
-(kicad_sch
-	(version 20260306)
-	(generator "eeschema")
-	(generator_version "10.0")
-	(paper "A4")
-	(sheet_instances
-		(path "/"
-			(page "1")
-		)
-	)
-	(embedded_fonts no)
-)
