File: hardware/Smart-Metering/08_Communications.kicad_sch (KiCad schematic)
At the start: 0 parts

Commit message: Completa o esquemático: MCU, interface HMI e comunicações
05_Metrology_MCU: STM32F413RHT6 (símbolo oficial), mesma família da
plataforma de referência da biblioteca ADSW-PQ-CLS (NUCLEO-F413ZH).
SPI1 isolado para ADE9430/MCP3204, IRQ/DREADY/ZX em EXTI, CF1/CF2 em
timers, USART2 para a HMI, USART3 + DE para RS-485, USB FS, VBAT_SENSE,
estado do carregador, HSE 8 MHz, RTC com LSE 32,768 kHz e CR2032, SWD
de 10 pinos e LEDs de status e pulso.

07_HMI_Interface: conector J701 para a placa HMI (ESP32-P4), com +5V
protegido por PTC e UART/IRQ/EN com resistores de 33 Ω.

08_Communications: RS-485/Modbus isolada com ADM2587E (terminação por
jumper e TVS) e USB-C de serviço com CC de 5,1 kΩ, ESD USBLC6-2SC6 e
detecção de VBUS.

Gerador: direção dos labels pela orientação do pino, pinos empilhados
tratados como um ponto, flags de não conectado.
README e ARCHITECTURE atualizados com o estado completo.

Co-Authored-By: Claude Opus 5.5 <noreply@anthropic.com>
Claude-Session: https://claude.ai/code/session_012B8cVkhtjf3eg98UdpNCpf
Parts:
- added C801, C803: 10uF, Capacitor_SMD:C_0805_2012Metric, symbol SmartMetering:C_Vert
- added C802, C804: 100nF, Capacitor_SMD:C_0603_1608Metric, symbol SmartMetering:C_Vert
- added C805: 4.7nF, Capacitor_SMD:C_1206_3216Metric, symbol SmartMetering:C_Vert
- added D801, D802: SMAJ12CA, Diode_SMD:D_SMA, symbol SmartMetering:D_TVS_Bi
- added J801: RS485, TerminalBlock_Phoenix:TerminalBlock_Phoenix_MKDS-1,5-3-5.08_1x03_P5.08mm_Horizontal, symbol SmartMetering:Conn_01x03
- added J802: USB-C, Connector_USB:USB_C_Receptacle_GCT_USB4105-xx-A_16P_TopMnt_Horizontal, symbol Connector:USB_C_Receptacle_USB2.0_16P
- added JP801: TERM, Connector_PinHeader_2.54mm:PinHeader_1x02_P2.54mm_Vertical, symbol SmartMetering:Jumper_2
- added R801: 120R, Resistor_SMD:R_1206_3216Metric, symbol SmartMetering:R_Vert
- added R802, R803: 5.1k, Resistor_SMD:R_0603_1608Metric, symbol SmartMetering:R_Vert
- added R804: 1M, Resistor_SMD:R_0603_1608Metric, symbol SmartMetering:R_Vert
- added R805: 10k, Resistor_SMD:R_0603_1608Metric, symbol SmartMetering:R_Vert
- added R806: 20k, Resistor_SMD:R_0603_1608Metric, symbol SmartMetering:R_Vert
- added U801: ADM2587E, Package_SO:SOIC-20W_7.5x12.8mm_P1.27mm, symbol Interface_UART:ADM2587E
- added U802: USBLC6-2SC6, Package_TO_SOT_SMD:SOT-23-6, symbol Power_Protection:USBLC6-2SC6
Connections:
- new net +3V3: C801.1, C802.1, U801.2 (VCC), U801.8 (VCC)
- new net BUS_A: D801.1, J801.1, R801.1, U801.13 (Y), U801.18 (A)
- new net BUS_B: D802.1, J801.2, JP801.2, U801.15 (Z), U801.17 (B)
- new net CC1: J802.A5 (CC1), R802.1
- new net CC2: J802.B5 (CC2), R803.1
- new net GND_485: C803.2, C804.2, D801.2, D802.2, J801.3, U801.11 (GND2), U801.14 (GND2), U801.16 (GND2), U801.20 (GND2)
- new net GND_SYS: C801.2, C802.2, C805.2, J802.A1 (GND), J802.A12 (GND), J802.B1 (GND), J802.B12 (GND), R802.2, R803.2, R804.2, R806.2, U801.1 (GND1), U801.10 (GND1), U801.3 (GND1), U801.9 (GND1), U802.2 (GND)
- new net RS485_DE: U801.5 (~{RE}), U801.6 (DE)
- new net RS485_RX: U801.4 (RxD)
- new net RS485_TX: U801.7 (TxD)
- new net TERM: JP801.1, R801.2
- new net USB_DM: J802.A7 (D-), J802.B7 (D-), U802.3 (I/O2), U802.4 (I/O2)
- new net USB_DP: J802.A6 (D+), J802.B6 (D+), U802.1 (I/O1), U802.6 (I/O1)
- new net USB_SHIELD: C805.1, J802.SH (SHIELD), R804.1
- new net USB_VBUS_SENSE: R805.2, R806.1
- new net VBUS: J802.A4 (VBUS), J802.A9 (VBUS), J802.B4 (VBUS), J802.B9 (VBUS), R805.1, U802.5 (VBUS)
- new net VISO_485: C803.1, C804.1, U801.12 (Visoout), U801.19 (Visoin)
- no-connect marks 0 -> 2
Other:
- note added: "RS-485 / MODBUS RTU ISOLADA U801 ADM2587E: transceptor + isolação de sinal e alimentação (isoPower) em um só CI. Half-duplex: A=Y e B=Z unidos; DE e ~RE unidos em RS485_DE (alto = transmite). JP801 liga a terminação de 120 Ω nos extremos do barramento. D801/D802: surtos. GND_485 é isolado do GND_SYS: levar ao borne J801 para referência do barramento. USB-C DE SERVIÇO R802/R803 (5,1 kΩ) identifica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"
- company: (none) -> Smart-Metering
- title: (none) -> Communications - RS-485 and USB-C

Commit message: Revisão completa do esquemático e correções
Verificação automática sobre o netlist global (215 componentes, 176 nets):
sem pinos soltos, sem nets de alimentação sem fonte, sem saídas em
conflito e isolação íntegra (terras só se encontram nas barreiras
PS101, PS601, U601, U602 e U801).

Correções:
- footprint do ADE9430 inexistente na biblioteca KiCad trocado por
  QFN-40 6x6 (tamanho do pad exposto a confirmar);
- MISO do ADE9430 como tri-state (barramento compartilhado com MCP3204);
- PS101 com símbolo e footprint oficiais do IRM-10-5 (o símbolo genérico
  tinha AC/L e AC/N trocados);
- PWR_FLAG em HV_DC, HV_RTN, VBAT_RTC, VDDA, GND_485 e VIN_CHG;
- footprints para fusíveis, varistores, indutores e chave de energia;
- polarização de fail-safe opcional no RS-485 (R807/R808, DNP);
- notas de layout (retorno do AC/DC) e de firmware (VBUS no PA9).

Relatório com revisão por folha, orçamento de potência e pendências em
docs/REVISAO_ESQUEMATICO.md.

Co-Authored-By: Claude Opus 5.5 <noreply@anthropic.com>
Claude-Session: https://claude.ai/code/session_012B8cVkhtjf3eg98UdpNCpf
Parts:
- added R807, R808: 680R, Resistor_SMD:R_0603_1608Metric, symbol SmartMetering:R_Vert
Connections:
- net BUS_A: now also R807.2
- net BUS_B: now also R808.1
- net GND_485: now also R808.2
- net VISO_485: now also R807.1
Other:
- note added: "RS-485 / MODBUS RTU ISOLADA U801 ADM2587E: transceptor + isolação de sinal e alimentação (isoPower) em um só CI. Half-duplex: A=Y e B=Z unidos; DE e ~RE unidos em RS485_DE (alto = transmite). JP801 liga a terminação de 120 Ω nos extremos do barramento. D801/D802: surtos. R807/R808 (DNP): polarização de fail-safe, montar em um único nó do barramento se necessário. GND_485 é isolado do GND_SYS: lev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"
- note removed: "RS-485 / MODBUS RTU ISOLADA U801 ADM2587E: transceptor + isolação de sinal e alimentação (isoPower) em um só CI. Half-duplex: A=Y e B=Z unidos; DE e ~RE unidos em RS485_DE (alto = transmite). JP801 liga a terminação de 120 Ω nos extremos do barramento. D801/D802: surtos. GND_485 é isolado do GND_SYS: levar ao borne J801 para referência do barramento. USB-C DE SERVIÇO R802/R803 (5,1 kΩ) identifica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"
Changed lines of the file:
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@@
 		(comment 2 "RS-485 bus side referenced to GND_485 (isolated)")
 	)
-	(text "RS-485 / MODBUS RTU ISOLADA\nU801 ADM2587E: transceptor + isolação de sinal e alimentação (isoPower) em um só CI.\nHalf-duplex: A=Y e B=Z unidos; DE e ~RE unidos em RS485_DE (alto = transmite).\nJP801 liga a terminação de 120 Ω nos extremos do barramento. D801/D802: surtos.\nGND_485 é isolado do GND_SYS: levar ao borne J801 para referência do barramento.\n\nUSB-C DE SERVIÇO\nR802/R803 (5,1 kΩ) identificam o aparelho como dispositivo (recebe 5 V).\nVBUS vai para o carregador (folha 09) e para a detecção do MCU (PA9, divisor R805/R806).\nD+/D- direto ao USB FS do MCU com proteção ESD U802."
+	(text "RS-485 / MODBUS RTU ISOLADA\nU801 ADM2587E: transceptor + isolação de sinal e alimentação (isoPower) em um só CI.\nHalf-duplex: A=Y e B=Z unidos; DE e ~RE unidos em RS485_DE (alto = transmite).\nJP801 liga a terminação de 120 Ω nos extremos do barramento. D801/D802: surtos.\nR807/R808 (DNP): polarização de fail-safe, montar em um único nó do barramento se necessário.\nGND_485 é isolado do GND_SYS: levar ao borne J801 para referência do barramento.\n\nUSB-C DE SERVIÇO\nR802/R803 (5,1 kΩ) identificam o aparelho como dispositivo (recebe 5 V).\nVBUS vai para o carregador (folha 09) e para a detecção do MCU (PA9, divisor R805/R806).\nFirmware: desabilitar o VBUS sensing do OTG e ler PA9 como GPIO (o divisor entrega 3,3 V).\nD+/D- direto ao USB FS do MCU com proteção ESD U802."
 		(exclude_from_sim no)(at 180.34 101.6 0)
 		(effects (font (size 1.27 1.27)) (justify left top))
@@
 	)
 	(label "GND_485" (at 215.9 80.01 270)
+		(effects (font (size 1.27 1.27)) (justify right bottom))
+	)
+	(label "GND_485" (at 165.1 50.8 270)
+		(effects (font (size 1.27 1.27)) (justify right bottom))
+	)
+	(label "VISO_485" (at 228.6 46.99 90)
+		(effects (font (size 1.27 1.27)) (justify left bottom))
+	)
+	(label "BUS_A" (at 228.6 54.61 270)
+		(effects (font (size 1.27 1.27)) (justify right bottom))
+	)
+	(label "BUS_B" (at 241.3 46.99 90)
+		(effects (font (size 1.27 1.27)) (justify left bottom))
+	)
+	(label "GND_485" (at 241.3 54.61 270)
 		(effects (font (size 1.27 1.27)) (justify right bottom))
 	)
@@
 			)
 		)
+	)
+	(symbol
+		(lib_id "power:PWR_FLAG")
+		(at 165.1 50.8 0)
+		(unit 1)(body_style 1)
+		(exclude_from_sim no)(in_bom yes)(on_board yes)(in_pos_files yes)(dnp no)
+		(property "Reference" "#FLG801" (at 165.1 46.99 0) (effects (font (size 1.27 1.27))))
+		(property "Value" "PWR_FLAG" (at 165.1 48.26 0) (effects (font (size 1.27 1.27))))
+		(property "Footprint" "" (at 165.1 50.8 0) (effects (font (size 1.27 1.27)) (hide yes)))
+		(property "Datasheet" "" (at 165.1 50.8 0) (effects (font (size 1.27 1.27)) (hide yes)))
+		(property "Description" "" (at 165.1 50.8 0) (effects (font (size 1.27 1.27)) (hide yes)))
+		(pin "1")
+		(instances
+			(project "Smart-Metering"
+				(path "/5fa62d70-4279-48bb-8603-6bcc60fb353a/a10e1008-0008-4e08-9008-000000000008" (reference "#FLG801") (unit 1))
+			)
+		)
+	)
+	(symbol
+		(lib_id "SmartMetering:R_Vert")
+		(at 228.6 50.8 0)
+		(unit 1)(body_style 1)
+		(exclude_from_sim no)(in_bom yes)(on_board yes)(in_pos_files yes)(dnp yes)
+		(property "Reference" "R807" (at 231.14 49.53 0) (effects (font (size 1.27 1.27)) (justify left)))
+		(property "Value" "680R" (at 231.14 52.07 0) (effects (font (size 1.27 1.27)) (justify left)))
+		(property "Footprint" "Resistor_SMD:R_0603_1608Metric" (at 228.6 50.8 0) (effects (font (size 1.27 1.27)) (hide yes)))
+		(property "Datasheet" "" (at 228.6 50.8 0) (effects (font (size 1.27 1.27)) (hide yes)))
+		(property "Description" "Fail-safe bias A to VISO (DNP by default)" (at 228.6 50.8 0) (effects (font (size 1.27 1.27)) (hide yes)))
+		(pin "1")
+		(pin "2")
+		(instances
+			(project "Smart-Metering"
+				(path "/5fa62d70-4279-48bb-8603-6bcc60fb353a/a10e1008-0008-4e08-9008-000000000008" (reference "R807") (unit 1))
+			)
+		)
+	)
+	(symbol
+		(lib_id "SmartMetering:R_Vert")
+		(at 241.3 50.8 0)
+		(unit 1)(body_style 1)
+		(exclude_from_sim no)(in_bom yes)(on_board yes)(in_pos_files yes)(dnp yes)
+		(property "Reference" "R808" (at 243.84 49.53 0) (effects (font (size 1.27 1.27)) (justify left)))
+		(property "Value" "680R" (at 243.84 52.07 0) (effects (font (size 1.27 1.27)) (justify left)))
+		(property "Footprint" "Resistor_SMD:R_0603_1608Metric" (at 241.3 50.8 0) (effects (font (size 1.27 1.27)) (hide yes)))
+		(property "Datasheet" "" (at 241.3 50.8 0) (effects (font (size 1.27 1.27)) (hide yes)))
+		(property "Description" "Fail-safe bias B to GND_485 (DNP by default)" (at 241.3 50.8 0) (effects (font (size 1.27 1.27)) (hide yes)))
+		(pin "1")
+		(pin "2")
+		(instances
+			(project "Smart-Metering"
+				(path "/5fa62d70-4279-48bb-8603-6bcc60fb353a/a10e1008-0008-4e08-9008-000000000008" (reference "R808") (unit 1))
+			)
+		)
