File: hardware/Smart-Metering/01_Power_Input.kicad_sch (KiCad schematic)
At the start: 17 parts, among them J101 AUX L N

Commit message: Resolve as pendências da revisão do esquemático
P1  ADE9430: footprint VQFN-40 6x6 com EP de 4,15 mm, compatível com as
    variantes CP-40 de 6x6 mm (EP de 3,9 a 4,7 mm).
P2  Confirmado no datasheet: MISO solto com SS alto (pull-up de 100 kΩ)
    e NC1/NC2 em GND, como já estava.
P3  J301-J304: headers JST PH de 4 vias cabeados até conectores M8
    fêmea de painel (à prova de toque).
P4  PS601 -> U606 ADuM6000 (isoPower 5 kVrms, símbolo oficial).
P5  PS101 -> RAC20-05SK/277 (85-305 VAC, 120-430 VDC, 20 W); fusíveis
    T500mA, R101 3 W, C101 10 uF/450 V; entrada do BQ25895 a 3 A.
P7  TPS61089 -> TPS61022 (compensação interna, sem valores a ajustar).
P8  Placa EV alimentada pelos pinos 5 V do J1 (nota na folha 07).
P9  EEPROM de calibração 24LC64 no I2C1.
P10 Labels globais de uma só folha convertidos em locais.

Verificação: 223 componentes, nenhum pino solto, nenhuma net sem fonte,
nenhum conflito de saída, isolação íntegra, todos os footprints
existentes na biblioteca oficial do KiCad.

Co-Authored-By: Claude Opus 5.5 <noreply@anthropic.com>
Claude-Session: https://claude.ai/code/session_012B8cVkhtjf3eg98UdpNCpf
Parts:
- C101: value 4.7uF 450V -> 10uF 450V; footprint Capacitor_THT:CP_Radial_D8.0mm_P3.50mm -> Capacitor_THT:CP_Radial_D10.0mm_P5.00mm
- F101, F102, F103, F104: value T250mA 500VAC -> T500mA 500VAC
- PS101: value IRM-10-5 -> RAC20-05SK/277; footprint Converter_ACDC:Converter_ACDC_MeanWell_IRM-10-xx_THT -> Converter_ACDC:Converter_ACDC_Recom_RAC20-xxSK_THT; symbol Converter_ACDC:IRM-10-5 -> Converter_ACDC:RAC20-05SK
- R101: value 22R 2W -> 22R 3W; footprint Resistor_THT:R_Axial_DIN0414_L11.9mm_D4.5mm_P15.24mm_Horizontal -> Resistor_THT:R_Axial_DIN0617_L17.0mm_D6.0mm_P20.32mm_Horizontal
Connections:
- net GND_SYS: now also PS101.4 (-Vout); no longer PS101.3 (-Vo)
- net VIN_ACDC: now also PS101.5 (+Vout); no longer PS101.4 (+Vo)
Other:
- note added: "PS101: RECOM RAC20-05SK/277, AC/DC isolado (reforçado), 5 V / 4 A; 85-305 VAC / 120-430 VDC. Ele é a barreira de isolação entre a rede e o domínio seguro (GND_SYS). Confirmar isolação e categoria de sobretensão do módulo para CAT III 300 V; a proteção de surto vem dos varistores (folha 02 e RV101) e de R101 (fusível, limita inrush). R101 (3 W) e C101 (10 uF): limitam a partida e filtram o ripple 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"
- note removed: "PS101: módulo AC/DC isolado (reforçado), 5 V / 2 A, aceita entrada CC 120-370 V. Ele é a barreira de isolação entre a rede e o domínio seguro (GND_SYS). Confirmar isolação e categoria de sobretensão do módulo para CAT III 300 V; a proteção de surto vem dos varistores (folha 02 e RV101) e de R101 (fusível, limita inrush). R101 e C101: limitam a corrente de partida e filtram o ripple do retificador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"
Changed lines of the file:
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@@
 		(effects (font (size 1.27 1.27)) (justify left top))
 	)
-	(text "PS101: módulo AC/DC isolado (reforçado), 5 V / 2 A, aceita entrada CC 120-370 V.\nEle é a barreira de isolação entre a rede e o domínio seguro (GND_SYS).\nConfirmar isolação e categoria de sobretensão do módulo para CAT III 300 V;\na proteção de surto vem dos varistores (folha 02 e RV101) e de R101 (fusível, limita inrush).\nR101 e C101: limitam a corrente de partida e filtram o ripple do retificador de meia onda.\n\nPotência: 10 W cobre o sistema (~4,5 W) + carga da bateria (~3,8 W).\nPS101 usa o símbolo e o footprint oficiais do IRM-10-5 (biblioteca KiCad).\nHV_RTN: levar em trilha própria até o borne do neutro, sem passar pelo plano GND\nmetrológico, para o ruído do conversor não chegar ao ADE9430.\n\nLAYOUT: todo este bloco está no potencial da rede. Manter distâncias de isolação\nentre o barramento HV, os retornos e o lado de saída (GND_SYS) do PS101."
+	(text "PS101: RECOM RAC20-05SK/277, AC/DC isolado (reforçado), 5 V / 4 A; 85-305 VAC / 120-430 VDC.\nEle é a barreira de isolação entre a rede e o domínio seguro (GND_SYS).\nConfirmar isolação e categoria de sobretensão do módulo para CAT III 300 V;\na proteção de surto vem dos varistores (folha 02 e RV101) e de R101 (fusível, limita inrush).\nR101 (3 W) e C101 (10 uF): limitam a partida e filtram o ripple do retificador de meia onda.\n\nPotência: 20 W cobre o sistema (~5,2 W) + carga da bateria (~4,7 W) com folga.\nPS101 usa o símbolo/footprint oficiais do RAC20-05SK (a variante /277 tem o mesmo encapsulamento:\nconfirmar com a RECOM). Margem: 264 VAC (+20 %) = 373 Vpk, dentro dos 430 VDC.\nHV_RTN: levar em trilha própria até o borne do neutro, sem passar pelo plano GND\nmetrológico, para o ruído do conversor não chegar ao ADE9430.\n\nLAYOUT: todo este bloco está no potencial da rede. Manter distâncias de isolação\nentre o barramento HV, os retornos e o lado de saída (GND_SYS) do PS101."
 		(exclude_from_sim no)(at 200.66 88.9 0)
 		(effects (font (size 1.27 1.27)) (justify left top))
@@
 		(exclude_from_sim no)(in_bom yes)(on_board yes)(in_pos_files yes)(dnp no)
 		(property "Reference" "F101" (at 63.5 48.26 0) (effects (font (size 1.27 1.27))))
-		(property "Value" "T250mA 500VAC" (at 63.5 53.34 0) (effects (font (size 1.27 1.27))))
+		(property "Value" "T500mA 500VAC" (at 63.5 53.34 0) (effects (font (size 1.27 1.27))))
 		(property "Footprint" "Fuse:Fuseholder_Clip-5x20mm_Littelfuse_111_Inline_P20.00x5.00mm_D1.05mm_Horizontal" (at 63.5 50.8 0) (effects (font (size 1.27 1.27)) (hide yes)))
 		(property "Datasheet" "" (at 63.5 50.8 0) (effects (font (size 1.27 1.27)) (hide yes)))
@@
 		(exclude_from_sim no)(in_bom yes)(on_board yes)(in_pos_files yes)(dnp no)
 		(property "Reference" "F102" (at 63.5 60.96 0) (effects (font (size 1.27 1.27))))
-		(property "Value" "T250mA 500VAC" (at 63.5 66.04 0) (effects (font (size 1.27 1.27))))
+		(property "Value" "T500mA 500VAC" (at 63.5 66.04 0) (effects (font (size 1.27 1.27))))
 		(property "Footprint" "Fuse:Fuseholder_Clip-5x20mm_Littelfuse_111_Inline_P20.00x5.00mm_D1.05mm_Horizontal" (at 63.5 63.5 0) (effects (font (size 1.27 1.27)) (hide yes)))
 		(property "Datasheet" "" (at 63.5 63.5 0) (effects (font (size 1.27 1.27)) (hide yes)))
@@
 		(exclude_from_sim no)(in_bom yes)(on_board yes)(in_pos_files yes)(dnp no)
 		(property "Reference" "F103" (at 63.5 73.66 0) (effects (font (size 1.27 1.27))))
-		(property "Value" "T250mA 500VAC" (at 63.5 78.74 0) (effects (font (size 1.27 1.27))))
+		(property "Value" "T500mA 500VAC" (at 63.5 78.74 0) (effects (font (size 1.27 1.27))))
 		(property "Footprint" "Fuse:Fuseholder_Clip-5x20mm_Littelfuse_111_Inline_P20.00x5.00mm_D1.05mm_Horizontal" (at 63.5 76.2 0) (effects (font (size 1.27 1.27)) (hide yes)))
 		(property "Datasheet" "" (at 63.5 76.2 0) (effects (font (size 1.27 1.27)) (hide yes)))
@@
 		(exclude_from_sim no)(in_bom yes)(on_board yes)(in_pos_files yes)(dnp yes)
 		(property "Reference" "F104" (at 63.5 99.06 0) (effects (font (size 1.27 1.27))))
-		(property "Value" "T250mA 500VAC" (at 63.5 104.14 0) (effects (font (size 1.27 1.27))))
+		(property "Value" "T500mA 500VAC" (at 63.5 104.14 0) (effects (font (size 1.27 1.27))))
 		(property "Footprint" "Fuse:Fuseholder_Clip-5x20mm_Littelfuse_111_Inline_P20.00x5.00mm_D1.05mm_Horizontal" (at 63.5 101.6 0) (effects (font (size 1.27 1.27)) (hide yes)))
 		(property "Datasheet" "" (at 63.5 101.6 0) (effects (font (size 1.27 1.27)) (hide yes)))
@@
 		(exclude_from_sim no)(in_bom yes)(on_board yes)(in_pos_files yes)(dnp no)
 		(property "Reference" "R101" (at 100.33 99.06 0) (effects (font (size 1.27 1.27))))
-		(property "Value" "22R 2W" (at 100.33 104.14 0) (effects (font (size 1.27 1.27))))
-		(property "Footprint" "Resistor_THT:R_Axial_DIN0414_L11.9mm_D4.5mm_P15.24mm_Horizontal" (at 100.33 101.6 0) (effects (font (size 1.27 1.27)) (hide yes)))
+		(property "Value" "22R 3W" (at 100.33 104.14 0) (effects (font (size 1.27 1.27))))
+		(property "Footprint" "Resistor_THT:R_Axial_DIN0617_L17.0mm_D6.0mm_P20.32mm_Horizontal" (at 100.33 101.6 0) (effects (font (size 1.27 1.27)) (hide yes)))
 		(property "Datasheet" "" (at 100.33 101.6 0) (effects (font (size 1.27 1.27)) (hide yes)))
-		(property "Description" "Inrush limiter, fusible flameproof wirewound, 2 W" (at 100.33 101.6 0) (effects (font (size 1.27 1.27)) (hide yes)))
+		(property "Description" "Inrush limiter, fusible flameproof wirewound, 3 W" (at 100.33 101.6 0) (effects (font (size 1.27 1.27)) (hide yes)))
 		(pin "1")
 		(pin "2")
@@
 		(exclude_from_sim no)(in_bom yes)(on_board yes)(in_pos_files yes)(dnp no)
 		(property "Reference" "C101" (at 111.76 104.14 0) (effects (font (size 1.27 1.27)) (justify right)))
-		(property "Value" "4.7uF 450V" (at 111.76 106.68 0) (effects (font (size 1.27 1.27)) (justify right)))
-		(property "Footprint" "Capacitor_THT:CP_Radial_D8.0mm_P3.50mm" (at 114.3 104.14 0) (effects (font (size 1.27 1.27)) (hide yes)))
+		(property "Value" "10uF 450V" (at 111.76 106.68 0) (effects (font (size 1.27 1.27)) (justify right)))
+		(property "Footprint" "Capacitor_THT:CP_Radial_D10.0mm_P5.00mm" (at 114.3 104.14 0) (effects (font (size 1.27 1.27)) (hide yes)))
 		(property "Datasheet" "" (at 114.3 104.14 0) (effects (font (size 1.27 1.27)) (hide yes)))
 		(property "Description" "HV bus capacitor, 105 °C" (at 114.3 104.14 0) (effects (font (size 1.27 1.27)) (hide yes)))
@@
 	)
 	(symbol
-		(lib_id "Converter_ACDC:IRM-10-5")
+		(lib_id "Converter_ACDC:RAC20-05SK")
 		(at 139.7 104.14 0)
 		(unit 1)(body_style 1)
 		(exclude_from_sim no)(in_bom yes)(on_board yes)(in_pos_files yes)(dnp no)
 		(property "Reference" "PS101" (at 139.7 96.52 0) (effects (font (size 1.27 1.27))))
-		(property "Value" "IRM-10-5" (at 139.7 99.06 0) (effects (font (size 1.27 1.27))))
-		(property "Footprint" "Converter_ACDC:Converter_ACDC_MeanWell_IRM-10-xx_THT" (at 139.7 104.14 0) (effects (font (size 1.27 1.27)) (hide yes)))
+		(property "Value" "RAC20-05SK/277" (at 139.7 99.06 0) (effects (font (size 1.27 1.27))))
+		(property "Footprint" "Converter_ACDC:Converter_ACDC_Recom_RAC20-xxSK_THT" (at 139.7 104.14 0) (effects (font (size 1.27 1.27)) (hide yes)))
 		(property "Datasheet" "" (at 139.7 104.14 0) (effects (font (size 1.27 1.27)) (hide yes)))
-		(property "Description" "AC/DC 5 V 2 A, 85-264 VAC / 120-370 VDC input, reinforced (Mean Well IRM-10-5)" (at 139.7 104.14 0) (effects (font (size 1.27 1.27)) (hide yes)))
-		(pin "1")
-		(pin "2")
-		(pin "3")
+		(property "Description" "AC/DC 5 V 4 A 20 W, reinforced; /277 variant: 85-305 VAC, 120-430 VDC (confirm with RECOM)" (at 139.7 104.14 0) (effects (font (size 1.27 1.27)) (hide yes)))
+		(pin "1")
+		(pin "2")
 		(pin "4")
-		(instances
-			(project "Smart-Metering"
+		(pin "5")
+		(instances
+			(project "Smart-Metering"
