File: hardware/Smart-Metering/09_Power_Supplies.kicad_sch (KiCad schematic)
At the start: 0 parts

Commit message: Alterações locais: folha 10 e ajustes nas folhas
Parts:
- added C30, C31: 2.2uF X7R 10V, Capacitor_SMD:C_0805_2012Metric, symbol SmartMetering:C_Vert
- added J1: 5V METROLOGY INPUT, Connector_PinHeader_2.54mm:PinHeader_1x02_P2.54mm_Vertical, symbol SmartMetering:Supply_2Pin
- added U2: TPS7A2033PDBVR, Package_TO_SOT_SMD:SOT-23-5, symbol SmartMetering:TPS7A2033PDBVR
Connections:
- new net +3V3_ADE: C31.2, U2.5 (OUT)
- new net +5V_MET_IN: C30.2, J1.1 (5V), U2.1 (IN), U2.3 (EN)
- new net GND: C30.1, C31.1, J1.2 (RETURN), U2.2 (GND)
- no-connect marks 0 -> 1
Other:
- note added: "LOCAL REGULATOR ONLY - input 5 V +/-5%, dedicated ADE9430 rail. J1 supplied externally; flags describe this explicit input contract. GND is mains-referenced through VN_SENSE. Isolation is NOT implemented here. Budget 50 mA for this rail; MCU/HMI require separate power budgeting. No direct mains energization until input protection and isolation are validated."
- title: (none) -> ADE9430 local 3.3 V supply
Changed lines of the file:
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@@
-(kicad_sch
-	(version 20260306)
-	(generator "eeschema")
-	(generator_version "10.0")
-	(paper "A4")
-	(sheet_instances
-		(path "/"
-			(page "1")
-		)
-	)
-	(embedded_fonts no)
-)
