File: hardware/Smart-Metering/Smart-Metering.kicad_sch (KiCad schematic)
At the start: 0 parts

Commit message: Cria arquitetura hierárquica inicial do Smart-Metering
Other:
- added sheet ADE9430 (04_ADE9430.kicad_sch)
- added sheet Communications (08_Communications.kicad_sch)
- added sheet Current Sensing (03_Current_Sensing.kicad_sch)
- added sheet HMI Interface (07_HMI_Interface.kicad_sch)
- added sheet Isolation (06_Isolation.kicad_sch)
- added sheet Metrology MCU (05_Metrology_MCU.kicad_sch)
- added sheet Power Input (01_Power_Input.kicad_sch)
- added sheet Power Supplies (09_Power_Supplies.kicad_sch)
- added sheet Voltage Sensing (02_Voltage_Sensing.kicad_sch)
Changed lines of the file:
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@@
 	(generator_version "10.0")
 	(paper "A4")
-	(sheet_instances
-		(path "/"
-			(page "1")
+	(sheet (at 20 30) (size 65 25)
+		(stroke (width 0.1524) (type solid))
+		(fill (color 0 0 0 0.0))
+		(property "Sheetname" "Power Input"
+			(at 20 29.2 0)
+			(effects (font (size 1.27 1.27)) (justify left bottom))
+		)
+		(property "Sheetfile" "01_Power_Input.kicad_sch"
+			(at 20 55.5 0)
+			(effects (font (size 1.27 1.27)) (justify left top))
+		)
+		(instances
+			(project "Smart-Metering"
+				(path "/5fa62d70-4279-48bb-8603-6bcc60fb353a" (page "2"))
+			)
 		)
 	)
+	(sheet (at 110 30) (size 65 25)
+		(stroke (width 0.1524) (type solid))
+		(fill (color 0 0 0 0.0))
+		(property "Sheetname" "Voltage Sensing"
+			(at 110 29.2 0)
+			(effects (font (size 1.27 1.27)) (justify left bottom))
+		)
+		(property "Sheetfile" "02_Voltage_Sensing.kicad_sch"
+			(at 110 55.5 0)
+			(effects (font (size 1.27 1.27)) (justify left top))
+		)
+		(instances
+			(project "Smart-Metering"
+				(path "/5fa62d70-4279-48bb-8603-6bcc60fb353a" (page "3"))
+			)
+		)
+	)
+	(sheet (at 200 30) (size 65 25)
+		(stroke (width 0.1524) (type solid))
+		(fill (color 0 0 0 0.0))
+		(property "Sheetname" "Current Sensing"
+			(at 200 29.2 0)
+			(effects (font (size 1.27 1.27)) (justify left bottom))
+		)
+		(property "Sheetfile" "03_Current_Sensing.kicad_sch"
+			(at 200 55.5 0)
+			(effects (font (size 1.27 1.27)) (justify left top))
+		)
+		(instances
+			(project "Smart-Metering"
+				(path "/5fa62d70-4279-48bb-8603-6bcc60fb353a" (page "4"))
+			)
+		)
+	)
+	(sheet (at 20 90) (size 65 25)
+		(stroke (width 0.1524) (type solid))
+		(fill (color 0 0 0 0.0))
+		(property "Sheetname" "ADE9430"
+			(at 20 89.2 0)
+			(effects (font (size 1.27 1.27)) (justify left bottom))
+		)
+		(property "Sheetfile" "04_ADE9430.kicad_sch"
+			(at 20 115.5 0)
+			(effects (font (size 1.27 1.27)) (justify left top))
+		)
+		(instances
+			(project "Smart-Metering"
+				(path "/5fa62d70-4279-48bb-8603-6bcc60fb353a" (page "5"))
+			)
+		)
+	)
+	(sheet (at 110 90) (size 65 25)
+		(stroke (width 0.1524) (type solid))
+		(fill (color 0 0 0 0.0))
+		(property "Sheetname" "Metrology MCU"
+			(at 110 89.2 0)
+			(effects (font (size 1.27 1.27)) (justify left bottom))
+		)
+		(property "Sheetfile" "05_Metrology_MCU.kicad_sch"
+			(at 110 115.5 0)
+			(effects (font (size 1.27 1.27)) (justify left top))
+		)
+		(instances
+			(project "Smart-Metering"
+				(path "/5fa62d70-4279-48bb-8603-6bcc60fb353a" (page "6"))
+			)
+		)
+	)
+	(sheet (at 200 90) (size 65 25)
+		(stroke (width 0.1524) (type solid))
+		(fill (color 0 0 0 0.0))
+		(property "Sheetname" "Isolation"
+			(at 200 89.2 0)
+			(effects (font (size 1.27 1.27)) (justify left bottom))
+		)
+		(property "Sheetfile" "06_Isolation.kicad_sch"
+			(at 200 115.5 0)
+			(effects (font (size 1.27 1.27)) (justify left top))
+		)
+		(instances
+			(project "Smart-Metering"
+				(path "/5fa62d70-4279-48bb-8603-6bcc60fb353a" (page "7"))
+			)
+		)
+	)
+	(sheet (at 20 150) (size 65 25)
+		(stroke (width 0.1524) (type solid))
+		(fill (color 0 0 0 0.0))
+		(property "Sheetname" "HMI Interface"
+			(at 20 149.2 0)
+			(effects (font (size 1.27 1.27)) (justify left bottom))
+		)
+		(property "Sheetfile" "07_HMI_Interface.kicad_sch"
+			(at 20 175.5 0)
+			(effects (font (size 1.27 1.27)) (justify left top))
+		)
+		(instances
+			(project "Smart-Metering"
+				(path "/5fa62d70-4279-48bb-8603-6bcc60fb353a" (page "8"))
+			)
+		)
+	)
+	(sheet (at 110 150) (size 65 25)
+		(stroke (width 0.1524) (type solid))
+		(fill (color 0 0 0 0.0))
+		(property "Sheetname" "Communications"
+			(at 110 149.2 0)
+			(effects (font (size 1.27 1.27)) (justify left bottom))
+		)
+		(property "Sheetfile" "08_Communications.kicad_sch"
+			(at 110 175.5 0)
+			(effects (font (size 1.27 1.27)) (justify left top))
+		)
+		(instances
+			(project "Smart-Metering"
+				(path "/5fa62d70-4279-48bb-8603-6bcc60fb353a" (page "9"))
+			)
+		)
+	)
+	(sheet (at 200 150) (size 65 25)
+		(stroke (width 0.1524) (type solid))
+		(fill (color 0 0 0 0.0))
+		(property "Sheetname" "Power Supplies"
+			(at 200 149.2 0)
+			(effects (font (size 1.27 1.27)) (justify left bottom))
+		)
+		(property "Sheetfile" "09_Power_Supplies.kicad_sch"
+			(at 200 175.5 0)
+			(effects (font (size 1.27 1.27)) (justify left top))
+		)
+		(instances
+			(project "Smart-Metering"
+				(path "/5fa62d70-4279-48bb-8603-6bcc60fb353a" (page "10"))
+			)
+		)
+	)
+	(sheet_instances
+		(path "/" (page "1"))
+	)
 	(embedded_fonts no)

Commit message: Alterações locais: folha 10 e ajustes nas folhas
Other:
- added sheet Battery Interface (10_Battery_Interface.kicad_sch)
Changed lines of the file:
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@@
 	(generator "eeschema")
 	(generator_version "10.0")
-	(paper "A4")
+	(paper "A3")
 	(sheet (at 20 30) (size 65 25)
 		(stroke (width 0.1524) (type solid))
@@
 		)
 	)
+	(sheet (at 300 30) (size 65 25) (stroke (width 0.1524) (type solid)) (fill (color 0 0 0 0.0)) (property "Sheetname" "Battery Interface" (at 300 29.2 0) (effects (font (size 1.27 1.27)) (justify left bottom))) (property "Sheetfile" "10_Battery_Interface.kicad_sch" (at 300 55.5 0) (effects (font (size 1.27 1.27)) (justify left top))) (instances (project "Smart-Metering" (path "/5fa62d70-4279-48bb-8603-6bcc60fb353a" (page "11")))))
 	(sheet_instances
 		(path "/" (page "1"))
